File: pcb/Nosumor.sch (EAGLE design)
At the start: 126 parts, among them IC1 STM32F722RET, J4 SJ-43515TS-SMT-EDGE, J5 CX90M-16P, J6 CX90M-16P, K1 CHERRY-MX, K2 CHERRY-MX, K3 KSC623J, K4 KSC623J, K5 KSC623J, Q1 ABM8W-12.0000MHZ, Q2 CX2016DB, Q3 FDY100PZ, Q4 FDY100PZ, Q5 FDY100PZ, Q6 FDY100PZ, U1 3.3V, U2 FT2232H-56Q-REEL, U3 3.3V, U4 24CW1280T-I/OT, U5 9DoF IMU, U6 3.3V, U7 USB3370, U8 TLV320AIC3256

Commit message: PCB revision 1.3 with USB Type-C, more datasheets
Parts:
- removed J5, J6: CX90M-16P, connector:CX90M-16P
- removed L3: 120OHM-500MA, Seeed-Inductor:SMD-FERRITE-CHIP-120-OHM-500MA(0603)
- removed TP11, TP3, TP7: TPB1,27, testpad:TPB1,27
- added C53, C54, C55: 100nf, Seeed-Capacitor:CERAMIC-100NF-25V-10%-X7R(0402)
- added R29: 2k7, Seeed-Resistor:SMD-RES-1K-5%-1/16W(0402)
- added R30: 0, Seeed-Resistor:SMD-RES-1K-5%-1/16W(0402)
- added R31, R32: 5k1, Seeed-Resistor:SMD-RES-1K-5%-1/16W(0402)
- added U9: TLV320AIC3256, ti:TLV320AIC3256
- C29: value 100n -> 4u7; device Seeed-Capacitor:CERAMIC-100NF-25V-10%-X7R(0402) -> Seeed-Capacitor:CERAMIC-1UF-6.3V-10%-X5R(0402)
- C30: value 12pf -> 100n; device Seeed-Capacitor:CERAMIC-12PF-50V-5%-NPO(0402) -> Seeed-Capacitor:CERAMIC-100NF-25V-10%-X7R(0402)
- C31: value 100n -> 12pf; device Seeed-Capacitor:CERAMIC-100NF-25V-10%-X7R(0402) -> Seeed-Capacitor:CERAMIC-12PF-50V-5%-NPO(0402)
- C33: device Seeed-Capacitor:CERAMIC-10NF-50V-10%-X7R(0402) -> Seeed-Capacitor:CERAMIC-100NF-25V-10%-X7R(0402)
- C34: value 4u7 -> 100n; device Seeed-Capacitor:CERAMIC-4.7UF-10V-10%-X5R(0603) -> Seeed-Capacitor:CERAMIC-10NF-50V-10%-X7R(0402)
- C35: device Seeed-Capacitor:CERAMIC-1UF-6.3V-10%-X5R(0402) -> Seeed-Capacitor:CERAMIC-4.7UF-10V-10%-X5R(0603)
- C36: value 100n -> 4u7; device Seeed-Capacitor:CERAMIC-100NF-25V-10%-X7R(0402) -> Seeed-Capacitor:CERAMIC-4.7UF-10V-10%-X5R(0603)
- C38: device Seeed-Capacitor:CERAMIC-4.7UF-10V-10%-X5R(0603) -> Seeed-Capacitor:CERAMIC-1UF-6.3V-10%-X5R(0402)
- C39: value 2u2 -> 100n; device rcl:C-EUC0603K -> Seeed-Capacitor:CERAMIC-100NF-25V-10%-X7R(0402)
- C40: value 100nf -> 4u7; device Seeed-Capacitor:CERAMIC-100NF-25V-10%-X7R(0402) -> Seeed-Capacitor:CERAMIC-4.7UF-10V-10%-X5R(0603)
- C41, C48: value 100nf -> 2u2; device Seeed-Capacitor:CERAMIC-100NF-25V-10%-X7R(0402) -> rcl:C-EUC0603K
- C43, C44: value 4u7 -> 100nf; device Seeed-Capacitor:CERAMIC-1UF-6.3V-10%-X5R(0402) -> Seeed-Capacitor:CERAMIC-100NF-25V-10%-X7R(0402)
- C46: value 100nf -> 4u7; device Seeed-Capacitor:CERAMIC-100NF-25V-10%-X7R(0402) -> Seeed-Capacitor:CERAMIC-1UF-6.3V-10%-X5R(0402)
- C47: value 2u2 -> 4u7; device rcl:C-EUC0603K -> Seeed-Capacitor:CERAMIC-1UF-6.3V-10%-X5R(0402)
- J3: value (none) -> CX90M-16P; device Wurth_Elektronik_Electromechanic_Input-Output_Connectors_rev16b:629105150521 -> connector:CX90M-16P
- R11: value 10K 1/16W -> 0; device Seeed-Resistor:SMD-RES-10K-1%-1/16W(0402) -> Seeed-Resistor:SMD-RES-1K-5%-1/16W(0402)
- R12: value 100R -> 10K 1/16W; device Seeed-Resistor:SMD-RES-330R-1%-1/16W(0402) -> Seeed-Resistor:SMD-RES-10K-1%-1/16W(0402)
- R15: value 27R -> 100R
- R20: value 10R -> 27R
- R21: value 10K 1/16W -> 10R; device Seeed-Resistor:SMD-RES-10K-1%-1/16W(0402) -> Seeed-Resistor:SMD-RES-330R-1%-1/16W(0402)
- R27: value 20K -> 10K 1/16W; device Seeed-Resistor:SMD-RES-1K-5%-1/16W(0402) -> Seeed-Resistor:SMD-RES-10K-1%-1/16W(0402)
- R28: value 2k7 -> 20K
- U3: value 3.3V -> 1.8V
- U7: value USB3370 -> 1.8V; device microchip:USB3370 -> SparkFun-IC-Power:V_REG_AP2112K-3.3V
- U8: value TLV320AIC3256 -> USB3370; device ti:TLV320AIC3256 -> microchip:USB3370
Connections:
- net N$43 renamed DBG_DP
- net N$51 renamed DBG_DM
- removed net N$14: J4.4, L3.1, U8.GND_SENSE
- removed net N$2: R16.2, U8.DIN/MFP1
- removed net N$22: R17.2, U8.BCLK
- removed net N$3: R18.2, U8.DOUT/MFP2
- removed net N$33: C43.2, U7.VDD33, U7.VDDIO
- removed net N$36: C44.2, U7.VDD18
- removed net N$40: R20.2, U8.MCLK
- removed net N$7: R15.2, U8.GPIO/MFP5
- new net AGND: C38.1, C41.2, C43.1, C44.1, C50.2, C53.2, C54.2, J4.4, R11.2, R30.2, U9.AVSS, U9.PAD
- new net AIC_BCLK_R: R18.2, U9.BCLK
- new net AIC_DIN_R: R17.2, U9.DIN/MFP1
- new net AIC_DOUT_R: R19.2, U9.DOUT/MFP2
- new net AIC_GPIO_R: R16.2, U9.GPIO/MFP5
- new net AIC_MCLK_R: R21.2, U9.MCLK
- new net AIC_WCLK_R: R20.2, U9.WCLK
- new net AVDD: C38.2, C43.2, C54.1, U7.OUT, U9.AVDD, U9.DRVDD_HP
- new net N$10: C51.1, U9.IN3_L
- new net VUSB18: C46.2, U8.VDD18
- new net VUSB33: C45.2, U8.VDD33, U8.VDDIO
- net +1V8: now also C55.1, U9.DVDD, U9.DVDD_CP; no longer C41.2, C51.1, C52.1, U8.AVDD, U8.DRVDD_HP, U8.DVDD, U8.DVDD_CP
- net +3V3: now also C30.2, C37.2, C44.2, R12.2, R26.2, U9.IOVDD, U9.VSYS; no longer C29.2, C31.2, C40.2, R11.2, R21.2, U8.IOVDD, U8.VSYS
- net +5V: now also C29.2, C47.2, C49.2, C52.2, J3.VBUS, R28.2, U7.EN, U7.IN, U8.VBAT; no longer C45.2, C48.2, J3.1VCC, R27.2, U7.VBAT
- net AIC_BCLK: now also R18.1; no longer R17.1
- net AIC_DIN: now also R17.1; no longer R16.1
- net AIC_DOUT: now also R19.1; no longer R18.1
- net AIC_GPIO: now also R16.1; no longer R15.1
- net AIC_WCLK: now also R20.1; no longer R19.1
- net GND: now also C39.1, C46.1, C47.1, C49.1, C52.1, C55.2, J3.GND, J3.SHIELD, R11.1, R27.1, R31.1, R32.1, U8.GND, U9.DVSS, U9.DVSS_CP, U9.IOVSS, U9.SPI_SELECT; no longer C38.1, C39.2, C41.1, C43.1, C44.1, C48.1, C49.2, C50.2, C51.2, C52.2, J3.5GND, J3.GND@1, J3.GND@2, L3.2, R26.1, U8.AVSS, U8.DVSS, U8.DVSS_CP, U8.IOVSS, U8.PAD, U8.SPI_SELECT
- net I2C_SCL: now also U9.SCL/SSZ; no longer U8.SCL/SSZ
- net I2C_SDA: now also U9.SDA/MOSI; no longer U8.SDA/MOSI
- net KEY_1: now also R22.1; no longer R21.1
- net KEY_2: now also R23.1; no longer R22.1
- net KEY_3: now also R24.1; no longer R23.1
- net KEY_4: now also R25.1; no longer R24.1
- net KEY_5: now also R26.1; no longer R25.1
- net LED_B: now also R15.1; no longer R14.1
- net LED_G: now also R14.1; no longer R13.1
- net LED_R: now also R13.1; no longer R12.1
- net MCLK: now also R21.1, U8.REFCLK; no longer R20.1, U7.REFCLK
- net N$1: now also J3.CC1, R32.2; no longer R19.2, U8.WCLK
- net N$12: now also U9.HPR; no longer U8.HPR
- net N$13: now also U9.HPL; no longer U8.HPL
- net N$17: now also C51.2, R29.2, U9.MICDET; no longer C46.2, R28.2, U8.MICDET
- net N$18: now also R29.1, U9.MICBIAS; no longer R28.1, U8.MICBIAS
- net N$19: now also R30.1, U9.GND_SENSE; no longer C46.1, U8.IN1_L
- net N$20: now also C53.1, U9.IN1_L, U9.IN1_R, U9.IN2_L, U9.IN2_R, U9.IN3_R; no longer C49.1, U8.IN1_R, U8.IN2_L, U8.IN2_R, U8.IN3_L, U8.IN3_R
- net N$21: now also U9.REF; no longer U8.REF
- net N$23: now also C48.1, U9.FLY_N; no longer C47.1, U8.FLY_N
- net N$25: now also C48.2, U9.FLY_P; no longer C47.2, U8.FLY_P
- net N$26: now also C31.2; no longer C30.2
- net N$29: now also C40.2; no longer C38.2
- net N$32: now also R28.1, U8.VBUS; no longer R27.1, U7.VBUS
- net N$37: now also R27.2, U8.RBIAS; no longer R26.2, U7.RBIAS
- net N$38: now also C41.1, U9.VNEG; no longer C39.1, U8.VNEG
- net N$4: now also J3.D-, U8.DM; no longer J3.2D-, U7.DM
- net N$5: now also J3.D+, U8.DP; no longer J3.3D+, U7.DP
- net N$6: now also J3.CC2, R31.2; no longer J3.4ID, U7.ID
- net RGB_B: now also R15.2; no longer R14.2
- net RGB_G: now also R14.2; no longer R13.2
- net RGB_R: now also R13.2; no longer R12.2
- net SRST_N: now also C39.2, R12.1, U8.RESETB, U9.!RESET; no longer C37.2, R11.1, TP11.TP, U7.RESETB, U8.!RESET
- net SWCLK: no longer TP3.TP
- net SWDIO: no longer TP7.TP
- net ULPI_CLK: now also U8.CLKOUT; no longer U7.CLKOUT
- net ULPI_D0: now also U8.DATA0; no longer U7.DATA0
- net ULPI_D1: now also U8.DATA1; no longer U7.DATA1
- net ULPI_D2: now also U8.DATA2; no longer U7.DATA2
- net ULPI_D3: now also U8.DATA3; no longer U7.DATA3
- net ULPI_D4: now also U8.DATA4; no longer U7.DATA4
- net ULPI_D5: now also U8.DATA5; no longer U7.DATA5
- net ULPI_D6: now also U8.DATA6; no longer U7.DATA6
- net ULPI_D7: now also U8.DATA7; no longer U7.DATA7
- net ULPI_DIR: now also U8.DIR; no longer U7.DIR
- net ULPI_NXT: now also U8.NXT; no longer U7.NXT
- net ULPI_STP: now also U8.STP; no longer U7.STP
Other:
- note added: "Debug"
- note added: "Designer: Norman Zhi Revision: 1.3 Date: 2019-12-23"
- note added: "USB Mix"
- note removed: "Designer: Norman Zhi Revision: 1.2 Date: 2019-04-25"
- note removed: "UART & JTAG"
- note removed: "osu! USB Supplemental Box"
- moved on the sheet: C1, C13, C15, C20, C24, C29, C30, C31, C32, C33, C34, C35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
